Commit message: update xml and urdf

File: assets/zbot-v2-fixed/robot/robot.urdf (robot description, URDF)
Before this commit: robot z-bot2_fe_urdf, 20 links, 19 joints
Joints:
- joint left_elbow: type revolute -> fixed
- joint left_gripper: type revolute -> fixed
- joint left_shoulder_pitch: type revolute -> fixed
- joint left_shoulder_yaw: type revolute -> fixed
- joint right_elbow: type revolute -> fixed
- joint right_gripper: type revolute -> fixed
- joint right_shoulder_pitch: type revolute -> fixed
- joint right_shoulder_yaw: type revolute -> fixed

Commit message: adapt the orientationg

File: assets/zbot-v2-fixed/robot/robot.urdf (robot description, URDF)
Before this commit: robot z-bot2_fe_urdf, 20 links, 19 joints
Links:
- added link base, mass 0.001
Joints:
- added joint floating_base: type fixed, parent base, child Z-BOT2_MASTER-BODY-SKELETON, origin xyz=0 0 0 rpy=0 0 -1.5707963

Commit message: forward orientation

File: assets/zbot-v2-fixed/robot/robot.urdf (robot description, URDF)
Before this commit: robot z-bot2_fe_urdf, 21 links, 20 joints
Joints:
- joint floating_base: origin xyz=0 0 0 rpy=0 0 -1.5707963 -> xyz=0 0 0 rpy=0 0 1.5707963
